File: Dimmer_atmega328.brd (EAGLE design)
At the start: 100 x 60 mm, 38 parts, among them IC1 LM1117MP-3.3, IC2 7805TV, Q1 16MHz, SW1 Push Switch, T1 BT138-V, U2 ATMEGA328P_PDIP, X1 AC, X2 LOAD

Commit message: routing
single layer routing in progress
Parts:
- added R1: 330, resistor:0207/10
Connections:
- net N$16: now also R1.1
- net N$17: now also R1.2
Changed lines of the file:
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@@
 <setting verticaltext="up"/>
 </settings>
-<grid distance="1" unitdist="mil" unit="mil" style="lines" multiple="1" display="yes" altdistance="1" altunitdist="mm" altunit="mm"/>
+<grid distance="1" unitdist="mm" unit="mm" style="lines" multiple="1" display="yes" altdistance="1" altunitdist="mm" altunit="mm"/>
 <layers>
 <layer number="1" name="Top" color="4" fill="1" visible="yes" active="yes"/>
@@
 <attribute name="OC_FARNELL" value="unknown" x="9.5" y="49" size="1.778" layer="27" display="off"/>
 </element>
+<element name="R1" library="resistor" package="0207/10" value="330" x="115.8786" y="18.2258" rot="R180"/>
 </elements>
 <signals>
@@
 <wire x1="83.1554" y1="50.3574" x2="83.1554" y2="45.8376" width="1.778" layer="16"/>
 <wire x1="83.1554" y1="45.8376" x2="85.5" y2="43.493" width="1.778" layer="16"/>
+<contactref element="R1" pad="1"/>
+<wire x1="120.9586" y1="18.2258" x2="75.04" y2="38.54" width="0" layer="19" extent="1-1"/>
 </signal>
 <signal name="N$17">
@@
 <wire x1="63.31" y1="35.46" x2="66.88" y2="35.46" width="1.778" layer="16"/>
 <wire x1="66.88" y1="35.46" x2="69.96" y2="38.54" width="1.778" layer="16"/>
+<contactref element="R1" pad="2"/>
+<wire x1="110.7986" y1="18.2258" x2="63.31" y2="35.46" width="0" layer="19" extent="1-1"/>
 </signal>
 <signal name="N$18">

Commit message: external dimmer feedback
external dimmer feedback circuit added.
diode bridge with filter and devider circuit included in schematic
Parts:
- added C8: 0.1UF,400V, amit_rcl:C102-054X133
- added C9: 470UF,400V, amit_rcl:E7,5-18
- added D1, D2, D3, D4: 1N4007, amit_diode_1N4004:DO41-10
- added R3: 220K, amit_rcl:0207/10
- added R6: 3.9K, amit_rcl:0207/10
- added X4: (no value), amit_screw_terminal_23:W237-102
Connections:
- new net EXTERNAL_DIMMER_FEEDBACK: R3.1, R6.2, U2.23
- new net N$30: D1.A, D2.C, X4.1
- new net N$31: D3.A, D4.C, X4.2
- new net N$32: C8.1, C9.+, D1.C, D3.C, R3.2
- net GND: now also C8.2, C9.-, D2.A, D4.A, R6.1
Changed lines of the file:
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@@
 </element>
 <element name="R1" library="resistor" package="0207/10" value="330" x="115.8786" y="18.2258" rot="R180"/>
+<element name="X4" library="amit_screw_terminal_23" package="W237-102" value="" x="-6" y="9">
+<attribute name="OC_NEWARK" value="70K9898" x="-6" y="9" size="1.778" layer="27" display="off"/>
+<attribute name="MPN" value="237-102" x="-6" y="9" size="1.778" layer="27" display="off"/>
+<attribute name="MF" value="" x="-6" y="9" size="1.778" layer="27" display="off"/>
+<attribute name="OC_FARNELL" value="unknown" x="-6" y="9" size="1.778" layer="27" display="off"/>
+</element>
+<element name="D1" library="amit_diode_1N4004" package="DO41-10" value="1N4007" x="-4" y="-4"/>
+<element name="D2" library="amit_diode_1N4004" package="DO41-10" value="1N4007" x="-4" y="-11"/>
+<element name="D3" library="amit_diode_1N4004" package="DO41-10" value="1N4007" x="-4" y="-18"/>
+<element name="D4" library="amit_diode_1N4004" package="DO41-10" value="1N4007" x="-4" y="-25"/>
+<element name="C8" library="amit_rcl" package="C102-054X133" value="0.1UF,400V" x="-4" y="-33"/>
+<element name="C9" library="amit_rcl" package="E7,5-18" value="470UF,400V" x="-2" y="-45"/>
+<element name="R3" library="amit_rcl" package="0207/10" value="220K" x="-4" y="-58"/>
+<element name="R6" library="amit_rcl" package="0207/10" value="3.9K" x="-4" y="-63"/>
 </elements>
 <signals>
@@
 <wire x1="11.8872" y1="43.688" x2="11.8872" y2="47.6172" width="0.8128" layer="16"/>
 <wire x1="11.8872" y1="47.6172" x2="12" y2="47.73" width="0.8128" layer="16"/>
+<contactref element="D2" pad="A"/>
+<contactref element="D4" pad="A"/>
+<contactref element="C9" pad="-"/>
+<contactref element="C8" pad="2"/>
+<contactref element="R6" pad="1"/>
 <wire x1="25.69" y1="35.73" x2="33.31" y2="38.27" width="0" layer="19" extent="1-1"/>
 <wire x1="11.8872" y1="43.688" x2="19.5" y2="37.65" width="0" layer="19" extent="16-16"/>
 <wire x1="43.5" y1="25.08" x2="46.5342" y2="34.9852" width="0" layer="19" extent="16-16"/>
+<wire x1="1.08" y1="-11" x2="11.9794" y2="2.0668" width="0" layer="19" extent="16-16"/>
+<wire x1="1.08" y1="-25" x2="1.08" y2="-11" width="0" layer="19" extent="1-1"/>
+<wire x1="1.08" y1="-33" x2="1.08" y2="-25" width="0" layer="19" extent="1-1"/>
+<wire x1="1.81" y1="-45" x2="1.08" y2="-33" width="0" layer="19" extent="1-1"/>
+<wire x1="-9.08" y1="-63" x2="1.81" y2="-45" width="0" layer="19" extent="1-1"/>
 </signal>
 <signal name="VCC">
@@
 <signal name="N$29">
 </signal>
+<signal name="N$30">
+<contactref element="D1" pad="A"/>
+<contactref element="D2" pad="C"/>
+<contactref element="X4" pad="1"/>
+<wire x1="1.08" y1="-4" x2="-9.08" y2="-11" width="0" layer="19" extent="1-1"/>
+<wire x1="-8.5" y1="7.73" x2="1.08" y2="-4" width="0" layer="19" extent="1-1"/>
+</signal>
+<signal name="N$31">
+<contactref element="D3" pad="A"/>
+<contactref element="D4" pad="C"/>
+<contactref element="X4" pad="2"/>
+<wire x1="1.08" y1="-18" x2="-9.08" y2="-25" width="0" layer="19" extent="1-1"/>
+<wire x1="-3.5" y1="7.73" x2="1.08" y2="-18" width="0" layer="19" extent="1-1"/>
+</signal>
+<signal name="N$32">
+<contactref element="D1" pad="C"/>
+<contactref element="D3" pad="C"/>
+<contactref element="C9" pad="+"/>
+<contactref element="C8" pad="1"/>
+<contactref element="R3" pad="2"/>
+<wire x1="-5.81" y1="-45" x2="1.08" y2="-58" width="0" layer="19" extent="1-1"/>
+<wire x1="-9.08" y1="-33" x2="-5.81" y2="-45" width="0" layer="19" extent="1-1"/>
+<wire x1="-9.08" y1="-18" x2="-9.08" y2="-33" width="0" layer="19" extent="1-1"/>
+<wire x1="-9.08" y1="-4" x2="-9.08" y2="-18" width="0" layer="19" extent="1-1"/>
+</signal>
+<signal name="EXTERNAL_DIMMER_FEEDBACK">
+<contactref element="R3" pad="1"/>
+<contactref element="R6" pad="2"/>
+<contactref element="U2" pad="23"/>
+<wire x1="1.08" y1="-63" x2="-9.08" y2="-58" width="0" layer="19" extent="1-1"/>
+<wire x1="25.69" y1="33.19" x2="-9.08" y2="-58" width="0" layer="19" extent="1-1"/>
+</signal>
 </signals>
