File: Dimmer_atmega328.sch (EAGLE design)
At the start: 38 parts, among them IC1 LM1117MP-3.3, IC2 7805TV, Q1 16MHz, SW1 Push Switch, T1 BT138-V, U2 ATMEGA328P_PDIP, X1 AC, X2 LOAD

Commit message: routing
single layer routing in progress
Parts:
- added R1: 330, resistor:R-US_0207/10
Connections:
- net N$16: now also R1.1
- net N$17: now also R1.2
Changed lines of the file:
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@@
 <part name="C7" library="rcl" deviceset="CPOL-US" device="E2.5-6" value="10uf"/>
 <part name="X3" library="con-wago-500" deviceset="W237-102" device=""/>
+<part name="R1" library="resistor" deviceset="R-US_" device="0207/10" value="330"/>
 </parts>
 <sheets>
@@
 <instance part="R17" gate="G$1" x="35.56" y="53.34" rot="R270"/>
 <instance part="R18" gate="G$1" x="45.72" y="40.64" rot="R270"/>
+<instance part="R1" gate="G$1" x="78.74" y="40.64" rot="R180"/>
 </instances>
 <busses>
@@
 <wire x1="104.14" y1="20.32" x2="104.14" y2="40.64" width="0.1524" layer="91"/>
 <pinref part="R14" gate="G$1" pin="2"/>
+<pinref part="R1" gate="G$1" pin="1"/>
+<junction x="83.82" y="40.64"/>
 </segment>
 </net>
@@
 <pinref part="OK2" gate="-1" pin="A1"/>
 <wire x1="68.58" y1="50.8" x2="71.12" y2="50.8" width="0.1524" layer="91"/>
-</segment>
-</net>
+<wire x1="71.12" y1="50.8" x2="71.12" y2="40.64" width="0.1524" layer="91"/>
+<pinref part="R1" gate="G$1" pin="2"/>
+<wire x1="71.12" y1="40.64" x2="73.66" y2="40.64" width="0.1524" layer="91"/>
+</segment>
+</net>

Commit message: external dimmer feedback
external dimmer feedback circuit added.
diode bridge with filter and devider circuit included in schematic
Parts:
- added C8: 0.1UF,400V, amit_rcl:C-EU102-054X133
- added C9: 470UF,400V, amit_rcl:CPOL-USE7.5-18
- added D1, D2, D3, D4: 1N4007, amit_diode_1N4004:1N4004
- added R3: 220K, amit_rcl:R-US_0207/10
- added R6: 3.9K, amit_rcl:R-US_0207/10
- added X4: (no value), amit_screw_terminal_23:W237-102
Connections:
- new net EXTERNAL_DIMMER_FEEDBACK: R3.1, R6.2, U2.PC0(ADC0)
- new net N$30: D1.A, D2.C, X4-1.KL
- new net N$31: D3.A, D4.C, X4-2.KL
- new net N$32: C8.1, C9.+, D1.C, D3.C, R3.2
- net GND: now also C8.2, C9.-, D2.A, D4.A, R6.1
Changed lines of the file:
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@@
 <part name="X3" library="con-wago-500" deviceset="W237-102" device=""/>
 <part name="R1" library="resistor" deviceset="R-US_" device="0207/10" value="330"/>
+<part name="X4" library="amit_screw_terminal_23" deviceset="W237-102" device=""/>
+<part name="D1" library="amit_diode_1N4004" deviceset="1N4004" device="" value="1N4007"/>
+<part name="D2" library="amit_diode_1N4004" deviceset="1N4004" device="" value="1N4007"/>
+<part name="D3" library="amit_diode_1N4004" deviceset="1N4004" device="" value="1N4007"/>
+<part name="D4" library="amit_diode_1N4004" deviceset="1N4004" device="" value="1N4007"/>
+<part name="C8" library="amit_rcl" deviceset="C-EU" device="102-054X133" value="0.1UF,400V"/>
+<part name="C9" library="amit_rcl" deviceset="CPOL-US" device="E7.5-18" value="470UF,400V"/>
+<part name="R3" library="amit_rcl" deviceset="R-US_" device="0207/10" value="220K"/>
+<part name="R6" library="amit_rcl" deviceset="R-US_" device="0207/10" value="3.9K"/>
 </parts>
 <sheets>
@@
 </segment>
 </net>
+<net name="EXTERNAL_DIMMER_FEEDBACK" class="0">
+<segment>
+<pinref part="U2" gate="G$1" pin="PC0(ADC0)"/>
+<wire x1="93.98" y1="71.12" x2="109.22" y2="71.12" width="0.1524" layer="91"/>
+<label x="109.22" y="71.12" size="1.778" layer="95"/>
+</segment>
+</net>
 </nets>
 </sheet>
@@
 </segment>
 </net>
+</nets>
+</sheet>
+<sheet>
+<description>external dimmer feedback</description>
+<plain>
+</plain>
+<instances>
+<instance part="X4" gate="-1" x="30.48" y="53.34"/>
+<instance part="X4" gate="-2" x="30.48" y="38.1"/>
+<instance part="D1" gate="1" x="55.88" y="50.8" rot="R90"/>
+<instance part="D2" gate="1" x="55.88" y="38.1" rot="R90"/>
+<instance part="D3" gate="1" x="68.58" y="50.8" rot="R90"/>
+<instance part="D4" gate="1" x="68.58" y="38.1" rot="R90"/>
+<instance part="C8" gate="G$1" x="86.36" y="48.26"/>
+<instance part="C9" gate="G$1" x="78.74" y="45.72"/>
+<instance part="R3" gate="G$1" x="104.14" y="48.26" rot="R90"/>
+<instance part="R6" gate="G$1" x="104.14" y="35.56" rot="R90"/>
+</instances>
+<busses>
+</busses>
+<nets>
+<net name="N$30" class="0">
+<segment>
+<pinref part="D1" gate="1" pin="A"/>
+<pinref part="D2" gate="1" pin="C"/>
+<wire x1="55.88" y1="48.26" x2="55.88" y2="45.72" width="0.1524" layer="91"/>
+<pinref part="X4" gate="-1" pin="KL"/>
+<wire x1="55.88" y1="45.72" x2="55.88" y2="40.64" width="0.1524" layer="91"/>
+<wire x1="35.56" y1="53.34" x2="50.8" y2="53.34" width="0.1524" layer="91"/>
+<wire x1="50.8" y1="53.34" x2="50.8" y2="45.72" width="0.1524" layer="91"/>
+<wire x1="50.8" y1="45.72" x2="55.88" y2="45.72" width="0.1524" layer="91"/>
+<junction x="55.88" y="45.72"/>
+</segment>
+</net>
+<net name="N$31" class="0">
+<segment>
+<pinref part="D3" gate="1" pin="A"/>
+<pinref part="D4" gate="1" pin="C"/>
+<wire x1="68.58" y1="48.26" x2="68.58" y2="43.18" width="0.1524" layer="91"/>
+<pinref part="X4" gate="-2" pin="KL"/>
+<wire x1="68.58" y1="43.18" x2="68.58" y2="40.64" width="0.1524" layer="91"/>
+<wire x1="35.56" y1="38.1" x2="50.8" y2="38.1" width="0.1524" layer="91"/>
+<wire x1="50.8" y1="38.1" x2="50.8" y2="43.18" width="0.1524" layer="91"/>
+<wire x1="50.8" y1="43.18" x2="68.58" y2="43.18" width="0.1524" layer="91"/>
+<junction x="68.58" y="43.18"/>
+</segment>
+</net>
+<net name="N$32" class="0">
+<segment>
+<pinref part="D1" gate="1" pin="C"/>
+<pinref part="D3" gate="1" pin="C"/>
+<wire x1="55.88" y1="53.34" x2="68.58" y2="53.34" width="0.1524" layer="91"/>
+<wire x1="68.58" y1="53.34" x2="78.74" y2="53.34" width="0.1524" layer="91"/>
+<junction x="68.58" y="53.34"/>
+<pinref part="C9" gate="G$1" pin="+"/>
+<wire x1="78.74" y1="53.34" x2="86.36" y2="53.34" width="0.1524" layer="91"/>
+<wire x1="86.36" y1="53.34" x2="104.14" y2="53.34" width="0.1524" layer="91"/>
+<wire x1="78.74" y1="53.34" x2="78.74" y2="48.26" width="0.1524" layer="91"/>
+<pinref part="C8" gate="G$1" pin="1"/>
+<wire x1="86.36" y1="53.34" x2="86.36" y2="50.8" width="0.1524" layer="91"/>
+<pinref part="R3" gate="G$1" pin="2"/>
+</segment>
+</net>
+<net name="GND" class="0">
+<segment>
+<pinref part="D2" gate="1" pin="A"/>
+<wire x1="55.88" y1="35.56" x2="68.58" y2="35.56" width="0.1524" layer="91"/>
+<pinref part="D4" gate="1" pin="A"/>
+<junction x="68.58" y="35.56"/>
+<wire x1="68.58" y1="35.56" x2="78.74" y2="35.56" width="0.1524" layer="91"/>
+<pinref part="C9" gate="G$1" pin="-"/>
+<wire x1="78.74" y1="35.56" x2="86.36" y2="35.56" width="0.1524" layer="91"/>
+<wire x1="86.36" y1="35.56" x2="96.52" y2="35.56" width="0.1524" layer="91"/>
+<wire x1="78.74" y1="40.64" x2="78.74" y2="35.56" width="0.1524" layer="91"/>
+<pinref part="C8" gate="G$1" pin="2"/>
+<wire x1="86.36" y1="43.18" x2="86.36" y2="35.56" width="0.1524" layer="91"/>
+<pinref part="R6" gate="G$1" pin="1"/>
+<wire x1="104.14" y1="30.48" x2="96.52" y2="30.48" width="0.1524" layer="91"/>
+<wire x1="96.52" y1="30.48" x2="96.52" y2="35.56" width="0.1524" layer="91"/>
+<wire x1="104.14" y1="30.48" x2="116.84" y2="30.48" width="0.1524" layer="91"/>
+<label x="116.84" y="30.48" size="1.778" layer="95"/>
+</segment>
+</net>
+<net name="EXTERNAL_DIMMER_FEEDBACK" class="0">
+<segment>
+<pinref part="R3" gate="G$1" pin="1"/>
+<pinref part="R6" gate="G$1" pin="2"/>
+<wire x1="104.14" y1="40.64" x2="104.14" y2="43.18" width="0.1524" layer="91"/>
+<wire x1="104.14" y1="43.18" x2="114.3" y2="43.18" width="0.1524" layer="91"/>
+<label x="114.3" y="43.18" size="1.778" layer="95"/>
+</segment>
+</net>
